File: hardware/s85-build3-rom-serial/s85-build3-rom-serial.sch (KiCad schematic (older format))
At the start: 12 parts, among them SW1 Reset, U1 8085, U2 74LS573, U3 AT28C256, Y1 6.144MHz

Commit message: add more build step schematics and pics
Parts:
- added J1: FTDI, symbol Connector_Generic:Conn_01x06
Connections:
- net GND: now also J1.1 (Pin_1); no longer U1.5 (SID)
- net FTDI-RX: now reaches D1.2 (A), U1.4 (SOD)
- net FTDI-RX: now also J1.5 (Pin_5)
- new net FTDI-TX: J1.4 (Pin_4), U1.5 (SID)
- no-connect marks 9 -> 12
Other:
- note added: "Note: FTDI pin numbers\nmay differ from this"
- moved on the sheet: D1, R1, R2, SW1
Changed lines of the file:
@@
 encoding utf-8
 Sheet 1 1
-Title "Simple8085 ROM test LED"
-Date "2023-10-12"
+Title "Simple8085 ROM test serial"
+Date "2023-10-29"
 Rev "1.0"
 Comp "github.com/TomNisbet"
@@
 L Device:LED_Small D1
 U 1 1 652417E2
-P 4600 4350
-F 0 "D1" H 4700 4400 50  0000 C CNN
-F 1 "LED" H 4450 4400 50  0000 C CNN
-F 2 "" V 4600 4350 50  0001 C CNN
-F 3 "~" V 4600 4350 50  0001 C CNN
-	1    4600 4350
+P 4450 4350
+F 0 "D1" H 4550 4400 50  0000 C CNN
+F 1 "LED" H 4300 4400 50  0000 C CNN
+F 2 "" V 4450 4350 50  0001 C CNN
+F 3 "~" V 4450 4350 50  0001 C CNN
+	1    4450 4350
 	1    0    0    -1
 $EndComp
@@
 L power:GND #PWR06
 U 1 1 6524214B
-P 5250 4750
-F 0 "#PWR06" H 5250 4500 50  0001 C CNN
-F 1 "GND" H 5255 4577 50  0000 C CNN
-F 2 "" H 5250 4750 50  0001 C CNN
-F 3 "" H 5250 4750 50  0001 C CNN
-	1    5250 4750
+P 5250 4800
+F 0 "#PWR06" H 5250 4550 50  0001 C CNN
+F 1 "GND" H 5255 4627 50  0000 C CNN
+F 2 "" H 5250 4800 50  0001 C CNN
+F 3 "" H 5250 4800 50  0001 C CNN
+	1    5250 4800
 	1    0    0    -1
 $EndComp
@@
 L power:GND #PWR04
 U 1 1 65258AB5
-P 3850 4500
-F 0 "#PWR04" H 3850 4250 50  0001 C CNN
-F 1 "GND" H 3855 4327 50  0000 C CNN
-F 2 "" H 3850 4500 50  0001 C CNN
-F 3 "" H 3850 4500 50  0001 C CNN
-	1    3850 4500
+P 3700 4500
+F 0 "#PWR04" H 3700 4250 50  0001 C CNN
+F 1 "GND" H 3705 4327 50  0000 C CNN
+F 2 "" H 3700 4500 50  0001 C CNN
+F 3 "" H 3700 4500 50  0001 C CNN
+	1    3700 4500
 	-1   0    0    -1
 $EndComp
 Wire Wire Line
-	4500 4350 4200 4350
+	4350 4350 4050 4350
 $Comp
 L power:+5V #PWR07
@@
 L power:+5V #PWR010
 U 1 1 652694E6
-P 4150 5200
-F 0 "#PWR010" H 4150 5050 50  0001 C CNN
-F 1 "+5V" H 4165 5373 50  0000 C CNN
-F 2 "" H 4150 5200 50  0001 C CNN
-F 3 "" H 4150 5200 50  0001 C CNN
-	1    4150 5200
+P 3950 5200
+F 0 "#PWR010" H 3950 5050 50  0001 C CNN
+F 1 "+5V" H 3965 5373 50  0000 C CNN
+F 2 "" H 3950 5200 50  0001 C CNN
+F 3 "" H 3950 5200 50  0001 C CNN
+	1    3950 5200
 	-1   0    0    -1
 $EndComp
@@
 L Device:R_Small_US R2
 U 1 1 6526D40F
-P 4100 4350
-F 0 "R2" V 4050 4200 50  0000 C CNN
-F 1 "1K" V 4050 4500 50  0000 C CNN
-F 2 "" H 4100 4350 50  0001 C CNN
-F 3 "~" H 4100 4350 50  0001 C CNN
-	1    4100 4350
+P 3950 4350
+F 0 "R2" V 3900 4200 50  0000 C CNN
+F 1 "1K" V 3900 4500 50  0000 C CNN
+F 2 "" H 3950 4350 50  0001 C CNN
+F 3 "~" H 3950 4350 50  0001 C CNN
+	1    3950 4350
 	0    -1   1    0
 $EndComp
 Wire Wire Line
-	4000 4350 3850 4350
+	3850 4350 3700 4350
 Wire Wire Line
 	4750 2100 4650 2100
@@
 	4700 3800 4750 3800
 Wire Wire Line
-	3500 4050 4750 4050
+	3300 4050 4750 4050
 Wire Wire Line
 	4700 4150 4750 4150
 Wire Wire Line
-	4700 4350 4750 4350
+	4550 4350 4600 4350
 NoConn ~ 6000 3650
 Wire Wire Line
@@
 L Device:R_Small_US R1
 U 1 1 655859C5
-P 3900 5350
-F 0 "R1" V 3850 5200 50  0000 C CNN
-F 1 "10K" V 3850 5500 50  0000 C CNN
-F 2 "" H 3900 5350 50  0001 C CNN
-F 3 "~" H 3900 5350 50  0001 C CNN
-	1    3900 5350
+P 3700 5350
+F 0 "R1" V 3650 5200 50  0000 C CNN
+F 1 "10K" V 3650 5500 50  0000 C CNN
+F 2 "" H 3700 5350 50  0001 C CNN
+F 3 "~" H 3700 5350 50  0001 C CNN
+	1    3700 5350
 	0    1    1    0
 $EndComp
@@
 L Switch:SW_Push SW1
 U 1 1 65586A0A
-P 4500 5500
-F 0 "SW1" H 4500 5785 50  0000 C CNN
-F 1 "Reset" H 4500 5694 50  0000 C CNN
-F 2 "" H 4500 5700 50  0001 C CNN
-F 3 "~" H 4500 5700 50  0001 C CNN
-	1    4500 5500
+P 4250 5500
+F 0 "SW1" H 4250 5785 50  0000 C CNN
+F 1 "Reset" H 4250 5694 50  0000 C CNN
+F 2 "" H 4250 5700 50  0001 C CNN
+F 3 "~" H 4250 5700 50  0001 C CNN
+	1    4250 5500
 	-1   0    0    -1
 $EndComp
@@
 L power:GND #PWR05
 U 1 1 6558F852
-P 4750 5550
-F 0 "#PWR05" H 4750 5300 50  0001 C CNN
-F 1 "GND" H 4755 5377 50  0000 C CNN
-F 2 "" H 4750 5550 50  0001 C CNN
-F 3 "" H 4750 5550 50  0001 C CNN
-	1    4750 5550
-	1    0    0    -1
-$EndComp
-Wire Wire Line
-	4150 5200 4150 5350
-Wire Wire Line
-	4150 5350 4000 5350
-Wire Wire Line
-	4750 5550 4750 5500
-Wire Wire Line
-	4750 5500 4700 5500
-Wire Wire Line
-	3800 5350 3500 5350
-Connection ~ 3500 5350
-Wire Wire Line
-	3500 5350 3500 5500
-Wire Wire Line
-	3500 5500 4300 5500
-Text Notes 3850 5650 0    50   ~ 0
+P 4500 5550
+F 0 "#PWR05" H 4500 5300 50  0001 C CNN
+F 1 "GND" H 4505 5377 50  0000 C CNN
+F 2 "" H 4500 5550 50  0001 C CNN
+F 3 "" H 4500 5550 50  0001 C CNN
+	1    4500 5550
+	1    0    0    -1
+$EndComp
+Wire Wire Line
+	3950 5200 3950 5350
+Wire Wire Line
+	3950 5350 3800 5350
+Wire Wire Line
+	4500 5550 4500 5500
+Wire Wire Line
+	4500 5500 4450 5500
+Wire Wire Line
+	3600 5350 3300 5350
+Connection ~ 3300 5350
+Wire Wire Line
+	3300 5350 3300 5500
+Wire Wire Line
+	3300 5500 4050 5500
+Text Notes 3600 5650 0    50   ~ 0
 Reset Button
 Text Notes 7200 3300 0    50   ~ 0
@@
 Text Notes 2200 1400 0    50   ~ 0
 ROM 0000-7FFF\nand 8000-FFFF
-Wire Wire Line
-	3850 4350 3850 4450
-Wire Wire Line
-	4750 4450 3850 4450
-Connection ~ 3850 4450
-Wire Wire Line
-	3850 4450 3850 4500
 NoConn ~ 4700 3400
 Wire Wire Line
 	4700 3400 4750 3400
 Wire Wire Line
-	3500 4050 3500 5350
+	3300 4050 3300 5350
+Wire Wire Line
+	3700 4350 3700 4500
+$Comp
+L Connector_Generic:Conn_01x06 J1
+U 1 1 6540797A
+P 5950 5100
+F 0 "J1" H 6030 5092 50  0000 L CNN
+F 1 "FTDI" H 6030 5001 50  0000 L CNN
+F 2 "" H 5950 5100 50  0001 C CNN
+F 3 "~" H 5950 5100 50  0001 C CNN
+	1    5950 5100
+	1    0    0    -1
+$EndComp
+Wire Wire Line
+	4750 4450 4700 4450
+Wire Wire Line
+	4700 4450 4700 5200
+Wire Wire Line
+	4700 5200 5750 5200
+Wire Wire Line
+	4600 4350 4600 5300
+Wire Wire Line
+	4600 5300 5750 5300
+Connection ~ 4600 4350
+Wire Wire Line
+	4600 4350 4750 4350
+Text Label 5300 5300 0    50   ~ 0
+FTDI-RX
+Text Label 5300 5200 0    50   ~ 0
+FTDI-TX
+Wire Wire Line
+	5250 4750 5650 4750
+Wire Wire Line
+	5650 4750 5650 4900
+Wire Wire Line
+	5650 4900 5750 4900
+Connection ~ 5250 4750
+Wire Wire Line
+	5250 4750 5250 4800
+NoConn ~ 5750 5000
+NoConn ~ 5750 5100
+NoConn ~ 5750 5400
+Text Notes 5350 5650 0    50   ~ 0
+Note: FTDI pin numbers\nmay differ from this
 Wire Bus Line
 	6100 2800 6100 3550
